Commit message: changed the urdf and meshes folder

File: arduinobot_description/urdf/robotic_arm.urdf (robot description, URDF)
Before this commit: robot robotic_arm, 9 links, 8 joints
Joints:
- joint joint_1: axis -0.00078022 0.11635 0.99321 -> 0 1 0; limit lower=-3.142 upper=3.142 effort=300 velocity=3 -> lower=0 upper=3.142 effort=200 velocity=3; origin xyz=0 0 0.06 rpy=1.5708 0 0.45791 -> xyz=0 0 0.05 rpy=1.5708 0 0.45791
- joint joint_2: origin xyz=-0.1461 0.17286 0 rpy=-1.5708 0 -1.8957 -> xyz=-0.1461 0.18286 0 rpy=-1.5708 0 -1.8957
- joint joint_4: limit lower=-3.142 upper=3.142 effort=200 velocity=3 -> lower=0 upper=3.142 effort=200 velocity=3
- joint joint_5: limit lower=-1.57 upper=1.57 effort=200 velocity=3 -> lower=0 upper=3.142 effort=200 velocity=3
- joint joint_6: limit lower=-3.142 upper=3.142 effort=200 velocity=3 -> lower=0 upper=3.142 effort=200 velocity=3
- joint joint_7: axis 0 1 0 -> 0 -1 0; origin xyz=0 -0.06071 0.03614 rpy=0 1.1954 -1.5708 -> xyz=0 -0.06071 -0.03614 rpy=-3.1416 -1.4875 -1.5708
- joint joint_8: axis 0 -1 0 -> 0 1 0; origin xyz=0 -0.06071 0.03614 rpy=-3.1416 -1.4875 -1.5708 -> xyz=0 -0.06071 0.03614 rpy=0 1.1954 -1.5708

File: arduinobot_description/urdf/robotic_arm_core.xacro (robot description, xacro)
@@ -15,5 +15,5 @@
     <origin rpy = "0 0 0" xyz = "0.0 0.0 0.0"/>
   </joint>
-  <link
+<link
     name="base_link">
     <inertial>
@@ -59,5 +59,5 @@
     <inertial>
       <origin
-        xyz="-0.042602 0.076543 0.0034922"
+        xyz="-0.042602 0.086543 0.0034922"
         rpy="0 0 0" />
       <mass
@@ -99,5 +99,5 @@
     type="revolute">
     <origin
-      xyz="0 0 0.06"
+      xyz="0 0 0.05"
       rpy="1.5708 0 0.45791" />
     <parent
@@ -106,9 +106,9 @@
       link="link_1" />
     <axis
-      xyz="-0.00078022 0.11635 0.99321" />
-    <limit
-      lower="-3.142"
+      xyz="0 1 0" />
+    <limit
+      lower="0"
       upper="3.142"
-      effort="300"
+      effort="200"
       velocity="3" />
   </joint>
@@ -157,5 +157,5 @@
     type="revolute">
     <origin
-      xyz="-0.1461 0.17286 0"
+      xyz="-0.1461 0.18286 0"
       rpy="-1.5708 0 -1.8957" />
     <parent
@@ -282,5 +282,5 @@
       xyz="1 0 0" />
     <limit
-      lower="-3.142"
+      lower="0"
       upper="3.142"
       effort="200"
@@ -297,8 +297,8 @@
       <inertia
         ixx="0.00044952"
-        ixy="1.5247E-19"
-        ixz="2.7105E-20"
+        ixy="1.5924E-19"
+        ixz="1.3553E-20"
         iyy="0.00031694"
-        iyz="8.1315E-20"
+        iyz="7.4539E-20"
         izz="0.00044603" />
     </inertial>
@@ -340,6 +340,6 @@
       xyz="0 0 -1" />
     <limit
-      lower="-1.57"
-      upper="1.57"
+      lower="0"
+      upper="3.142"
       effort="200"
       velocity="3" />
@@ -355,8 +355,8 @@
       <inertia
         ixx="0.00011376"
-        ixy="-1.6305E-20"
-        ixz="1.1858E-20"
+        ixy="-1.1435E-20"
+        ixz="-1.6941E-21"
         iyy="0.00011418"
-        iyz="-1.8635E-20"
+        iyz="-7.6233E-21"
         izz="0.00010947" />
     </inertial>
@@ -398,5 +398,5 @@
       xyz="0 -1 0" />
     <limit
-      lower="-3.142"
+      lower="0"
       upper="3.142"
       effort="200"
@@ -447,6 +447,6 @@
     type="revolute">
     <origin
-      xyz="0 -0.06071 0.03614"
-      rpy="0 1.1954 -1.5708" />
+      xyz="0 -0.06071 -0.03614"
+      rpy="-3.1416 -1.4875 -1.5708" />
     <parent
       link="link_6" />
@@ -454,5 +454,5 @@
       link="gripper_1" />
     <axis
-      xyz="0 1 0" />
+      xyz="0 -1 0" />
     <limit
       lower="0"
@@ -465,5 +465,5 @@
     <inertial>
       <origin
-        xyz="-0.056383 6.5254E-05 0.057488"
+        xyz="0.015647 6.5254E-05 0.051476"
         rpy="0 0 0" />
       <mass
@@ -506,5 +506,5 @@
     <origin
       xyz="0 -0.06071 0.03614"
-      rpy="-3.1416 -1.4875 -1.5708" />
+      rpy="0 1.1954 -1.5708" />
     <parent
       link="link_6" />
@@ -512,5 +512,5 @@
       link="gripper_2" />
     <axis
-      xyz="0 -1 0" />
+      xyz="0 1 0" />
     <limit
       lower="0"
